File: Arduino_SMS_Cart_Programmer/Arduino_SMS_Cart_Programmer.kicad_sch (KiCad schematic)
At the start: 8 parts, among them J1 SEGA Master System Cartridge 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, U1 74HC595, U2 74HC595

Commit message: Added cart reset line connection.
Connections:
- net /RST: now reaches J1.46 (Pin_46)
- net /RST: now also A1.23 (A4)
Changed lines of the file:
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@@
+		)
+	)
+	(global_label "{slash}RST"
+		(shape output)
+		(at 87.63 99.06 0)
+		(fields_autoplaced yes)
+		(effects
+			(font
+				(size 1.27 1.27)
+			)
+			(justify left)
+		)
+		(property "Intersheetrefs" "${INTERSHEET_REFS}"
+			(at 95.3928 99.06 0)
+			(effects
+				(font
+					(size 1.27 1.27)
+				)
+				(justify left)
+				(hide yes)
+			)
 		)
 	)
@@
 			(effects
 				(font
+					(size 1.27 1.27)
+				)
+				(justify left)
+				(hide yes)
+			)
+		)
+	)
+	(global_label "{slash}RST"
+		(shape input)
+		(at 241.3 116.84 0)
+		(fields_autoplaced yes)
+		(effects
+			(font
+				(size 1.27 1.27)
+			)
+			(justify left)
+		)
+		(property "Intersheetrefs" "${INTERSHEET_REFS}"
+			(at 249.0628 116.84 0)
+			(effects
+				(font
